File: pcb/v3/hackapet_v2.kicad_pcb (KiCad board)
At the start: 2 copper layers, 56.8 x 66.2 mm, 40 parts, among them J1 Conn_01x07_Socket, J3 battery_holder, J4 USB_C_Receptacle_USB2.0_16P, J5 Conn_01x01_Socket, J6 Conn_01x01_Socket, J7 Conn_02x06_Counter_Clockwise, SW1 SW_Push, SW2 SW_Push, SW3 SW_Push, SW4 SW_SPDT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

Commit message: updated board
Parts:
- removed J7: Conn_02x06_Counter_Clockwise, Connector_PinSocket_2.54mm:PinSocket_2x06_P2.54mm_Vertical
- added BREAKOUT_PINS1: Conn_02x06_Odd_Even, Connector_PinHeader_2.54mm:PinHeader_2x06_P2.54mm_Vertical, F.Cu at (206.0, 87.4)
- added D8: S-LMBR340FT1G, Diode_SMD:D_0805_2012Metric, F.Cu at (213.2, 79.8)
- J3: footprint Battery:1022_batteryholder -> Battery:BatteryHolder_Keystone_2468_2xAAA
- moved J3 46.5 mm to (140.9, 61.3), turned to -90 degrees
- renumbered SW5 to BOOT1, J1 to DISPLAY_SSD1351, SW6 to RESET1
Connections:
- BOOT1 pad 1: GND -> -BATT
- C1 pad 1: GND -> -BATT
- C1 pad 2: +5V -> Net-(D2-K)
- C2 pad 2: GND -> -BATT
- C3 pad 1: GND -> -BATT
- C3 pad 2: +5V -> Net-(D2-K)
- C4 pad 2: GND -> -BATT
- C5 pad 2: GND -> -BATT
- C9 pad 2: GND -> -BATT
- D1 pad 1: +3V3 -> +BATT
- D2 pad 1: +5V -> Net-(D2-K)
- D3 pad 1: GND -> -BATT
- D4 pad 1: GND -> -BATT
- D5 pad 1: GND -> -BATT
- D7 pad 1: GND -> -BATT
- DISPLAY_SSD1351 pad 6: GND -> -BATT
- J4 pad A1: GND -> -BATT
- J4 pad A12: GND -> -BATT
- J4 pad B1: GND -> -BATT
- J4 pad B12: GND -> -BATT
- J4 pad S1: GND -> -BATT
- R4 pad 2: GND -> -BATT
- R5 pad 2: GND -> -BATT
- RESET1 pad 1: GND -> -BATT
- SW1 pad 1: GND -> -BATT
- SW2 pad 1: GND -> -BATT
- SW3 pad 1: GND -> -BATT
- U1 pad 1: GND -> -BATT
- U1 pad 3: +5V -> +BATT
- U2 pad 1: GND -> -BATT
- U2 pad 4: GND -> -BATT
- U3 pad 1: GND -> -BATT
- U3 pad 2: GND -> -BATT
- U3 pad 30: GND -> -BATT
- U3 pad 42: GND -> -BATT
- U3 pad 43: GND -> -BATT
- U3 pad 46: GND -> -BATT
- U3 pad 47: GND -> -BATT
- U3 pad 48: GND -> -BATT
- U3 pad 49: GND -> -BATT
- U3 pad 50: GND -> -BATT
- U3 pad 51: GND -> -BATT
- U3 pad 52: GND -> -BATT
- U3 pad 53: GND -> -BATT
- U3 pad 54: GND -> -BATT
- U3 pad 55: GND -> -BATT
- U3 pad 56: GND -> -BATT
- U3 pad 57: GND -> -BATT
- U3 pad 58: GND -> -BATT
- U3 pad 59: GND -> -BATT
- U3 pad 60: GND -> -BATT
- U3 pad 61: GND -> -BATT
- U3 pad 61_1: GND -> -BATT
- U3 pad 61_2: GND -> -BATT
- U3 pad 61_3: GND -> -BATT
- U3 pad 61_4: GND -> -BATT
- U3 pad 61_5: GND -> -BATT
- U3 pad 61_6: GND -> -BATT
- U3 pad 61_7: GND -> -BATT
- U3 pad 61_8: GND -> -BATT
- U3 pad 62: GND -> -BATT
- U3 pad 63: GND -> -BATT
- U3 pad 64: GND -> -BATT
- U3 pad 65: GND -> -BATT
Routing:
- net -BATT: track 0.00 -> 178.2 mm, vias 0 -> 56
- net GND: track 171.8 -> 0.00 mm, vias 54 -> 0
- net Net-(D2-K): track 0.00 -> 80.0 mm
- net +5V: track 64.8 -> 0.00 mm
- net +BATT: track 0.00 -> 16.3 mm
- net Net-(D1-A): track 24.7 -> 25.7 mm
- added copper zone on B.Cu, net -BATT
- added copper zone on F.Cu, net -BATT
- removed copper zone on B.Cu, net GND
- removed copper zone on F.Cu, net GND
