File: pcb/v3/hackapet_v2.kicad_sch (KiCad schematic)
At the start: 35 parts, among them J1 Conn_01x07_Socket, J3 battery_holder, J4 USB_C_Receptacle_USB2.0_16P, J5 Conn_01x01_Socket, J6 Conn_01x01_Socket, J7 Conn_02x06_Counter_Clockwise, SW1 SW_Push, SW2 SW_Push, SW3 SW_Push, SW4 SW_SPDT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

Commit message: moved batt to 3v3 regulator b/c no buck converter
Parts:
- removed J7: Conn_02x06_Counter_Clockwise, Connector_PinSocket_2.54mm:PinSocket_2x06_P2.54mm_Vertical, symbol Connector_Generic:Conn_02x06_Counter_Clockwise
- added BREAKOUT_PINS: Conn_02x06_Odd_Even, symbol Connector_Generic:Conn_02x06_Odd_Even
- added D8: S-LMBR340FT1G, Diode_SMD:D_0805_2012Metric, symbol Device:D
- renumbered SW5 to BOOT, J1 to DISPLAY_SSD1351, SW6 to RESET
Connections:
- net +3V3: now also BREAKOUT_PINS.10 (Pin_10); no longer D1.1 (K)
- net IO14: now also BREAKOUT_PINS.1 (Pin_1)
- net IO15: now also BREAKOUT_PINS.2 (Pin_2)
- net IO21: now also BREAKOUT_PINS.3 (Pin_3)
- net IO33: now also BREAKOUT_PINS.4 (Pin_4)
- net IO34: now also BREAKOUT_PINS.5 (Pin_5)
- net IO35: now also BREAKOUT_PINS.6 (Pin_6)
- net IO36: now also BREAKOUT_PINS.7 (Pin_7)
- net IO37: now also BREAKOUT_PINS.8 (Pin_8)
- net IO38: now also BREAKOUT_PINS.9 (Pin_9)
- net +5V: no longer names the net of C1.2, C3.2, D2.1 (K)
- net +5V: now also D8.2 (A); no longer U1.3 (VI)
- net GND renamed -BATT
- net -BATT: now also BREAKOUT_PINS.11 (Pin_11)
- new net +BATT: D1.1 (K), D8.1 (K), U1.3 (VI)
- no-connect marks 12 -> 13
Other:
- note removed: "can i connect this to the same clock"
- note removed: "is this 1.8v or 3v3"
- note removed: "this needs to be pulled down,, should i also connect to a pin??"
- moved on the sheet: BOOT, C1, C3, C4, C5, C9, D1, D2, D6, DISPLAY_SSD1351, J3, J4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

Commit message: updated board
Parts:
- renumbered BOOT to BOOT1, BREAKOUT_PINS to BREAKOUT_PINS1, RESET to RESET1
Changed lines of the file:
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@@
 (kicad_sch
-	(version 20241209)
+	(version 20250114)
 	(generator "eeschema")
-	(generator_version "8.99")
+	(generator_version "9.0")
 	(paper "A3")
 	(junction
@@
 		(on_board yes)
 		(dnp no)
-		(property "Reference" "RESET"
+		(property "Reference" "RESET1"
 			(at 167.64 86.3599 90)
 			(effects
@@
 			(project ""
 				(path "/090708b6-5b5c-47a2-9faf-b664b76dd2bb"
-					(reference "RESET")
+					(reference "RESET1")
 					(unit 1)
 				)
@@
 		(dnp no)
 		(fields_autoplaced yes)
-		(property "Reference" "BOOT"
+		(property "Reference" "BOOT1"
 			(at 198.12 43.18 0)
 			(effects
@@
 			(project "hackapet_v2"
 				(path "/090708b6-5b5c-47a2-9faf-b664b76dd2bb"
-					(reference "BOOT")
+					(reference "BOOT1")
 					(unit 1)
 				)
@@
 		(dnp no)
 		(fields_autoplaced yes)
-		(property "Reference" "BREAKOUT_PINS"
+		(property "Reference" "BREAKOUT_PINS1"
 			(at 262.89 106.68 0)
 			(effects
@@
 			(project ""
 				(path "/090708b6-5b5c-47a2-9faf-b664b76dd2bb"
-					(reference "BREAKOUT_PINS")
+					(reference "BREAKOUT_PINS1")
 					(unit 1)
 				)
